File: Hardware/SparkX_EZ_LiPo_Power.brd (EAGLE design)
At the start: 10.7 x 40.6 mm, 42 parts, among them J3 AVR_SPI_PROG_3X2TESTPOINTS, Q1 3.1A/30V/105mΩ, U1 ATTINY43_QFN20, U2 MCP73831, U3 3.3V, U4 MAX17048

Commit message: Partially routed
Parts:
- removed J2: (no value), SparkFun-Connectors:1X02_NO_SILK
- added BATT+: TEST-POINT3X4, SparkFun-Connectors:PAD.03X.04
- added FG_SDA: JUMPER-SMT_2_NC_TRACE_SILK, SparkFun-Jumpers:SMT-JUMPER_2_NC_TRACE_SILK
- moved AT_VCC 48.6 mm to (6.60, 12.7), turned to 180 degrees
- moved L1 47.0 mm to (7.81, 15.6), turned to 90 degrees
- moved PROC_PWR_EN 43.9 mm to (9.33, 3.62), flipped to the bottom, turned to 90 degrees
- moved C4 43.1 mm to (7.62, 29.2), turned to 270 degrees
- moved C5 41.9 mm to (8.83, 17.4)
- moved D3 40.5 mm to (4.00, 15.6)
- moved U1 40.1 mm to (5.33, 19.1)
- moved J3 39.6 mm to (5.33, 12.7)
- moved C7 38.4 mm to (1.59, 19.4), turned to 90 degrees
- moved C8 38.2 mm to (1.40, 17.3), turned to 180 degrees
- moved VIN 38.1 mm to (5.08, 17.8)
- moved C3 35.8 mm to (7.62, 7.87), turned to 90 degrees
- moved U3 35.3 mm to (5.33, 8.89), turned to 180 degrees
- moved R3 34.9 mm to (2.16, 26.9)
- moved C1 34.3 mm to (7.62, 9.91), turned to 270 degrees
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Connections:
- new net N$1: FG_SDA.1, U4.8
- net GND: no longer J2.2
- net SDA: now also FG_SDA.2; no longer U4.8
- net V_BATT: now also BATT+.1; no longer J2.1
Routing:
- net SCL: track 0.00 -> 68.2 mm, vias 0 -> 4
- net SDA: track 0.00 -> 57.1 mm, vias 0 -> 4
- net V_USB: track 0.00 -> 50.0 mm, vias 0 -> 3
- net PROC_PWR_EN: track 0.00 -> 41.6 mm, vias 0 -> 1
- net VIN: track 0.00 -> 37.6 mm, vias 0 -> 5
- net 3V3_EN: track 0.00 -> 26.8 mm
- net GND: track 0.00 -> 26.2 mm, vias 0 -> 17
- net 3.3V: track 0.00 -> 22.7 mm, vias 0 -> 4
- net V_BATT: track 0.00 -> 14.1 mm, vias 0 -> 1
- net AT_VCC: track 0.00 -> 11.4 mm
- net CHG_LED: track 0.00 -> 4.69 mm
- net N$1: track 0.00 -> 3.77 mm
- net N$21: track 0.00 -> 3.57 mm
- net N$2: track 0.00 -> 3.40 mm
- net N$20: track 0.00 -> 1.97 mm
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
Commit message: Freshly routed
Parts:
- moved U$20 21.6 mm to (5.33, 29.2)
- moved LOGO3 20.3 mm to (5.33, 23.5)
- moved LOGO2 9.01 mm to (1.71, 8.00), turned to 0 degrees
- moved U$1 2.96 mm to (6.73, 22.7), turned to 0 degrees
- moved AT_VCC 2.73 mm to (9.33, 12.7), turned to 270 degrees
- moved FG_SDA 2.02 mm to (8.38, 31.1)
- moved VIN 1.80 mm to (6.35, 19.1)
- moved 3V3_EN 1.27 mm to (3.81, 7.62)
- moved C4 0.63 mm to (8.00, 28.7), turned to 180 degrees
- moved C3 0.60 mm to (7.94, 7.37), turned to 0 degrees
- moved C7 0.51 mm to (1.14, 19.2)
- moved C8 0.25 mm to (1.40, 17.0)
- moved C1 0.13 mm to (7.75, 9.91)
Routing:
- net 3.3V: track 22.7 -> 77.6 mm, vias 4 -> 8
- net CS1: track 0.85 -> 43.5 mm
- net GPIO0: track 0.85 -> 43.3 mm
- net SCLK: track 0.84 -> 43.2 mm
- net CIPO: track 0.85 -> 43.2 mm
- net CS2: track 1.35 -> 43.3 mm
- net GPIO1: track 1.37 -> 43.3 mm
- net CS0: track 1.35 -> 43.2 mm
- net COPI: track 1.36 -> 43.2 mm
- net GND: track 26.2 -> 45.9 mm, vias 17 -> 39
- net AT_CIPO: track 0.76 -> 19.5 mm, vias 1 -> 2
- net !RESET!: track 0.00 -> 18.5 mm
- net V_BATT: track 14.1 -> 18.6 mm
- net 3V3_EN: track 26.8 -> 30.8 mm, vias 0 -> 1
- net SDA: track 57.1 -> 61.0 mm, vias 4 -> 5
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
Commit message: Ready for review
Parts:
- added U$2, U$3: (no value), output:EZ_POWER_LIPO0
- added U$4: (no value), output:#BATT##0
- added U$5: (no value), output:#VIN#0
- added U$6: (no value), output:#3V3_EN#0
- added U$7: (no value), output:#PROC_PWR#0
- added U$8: (no value), output:#AT_VCC#0
- added U$9: (no value), output:#FG_SDA#0
Routing:
- net GND: track 45.9 -> 89.4 mm, vias 39 -> 46
- net AT_CIPO: track 19.5 -> 20.7 mm
- net V_USB: track 50.0 -> 50.7 mm, vias 3 -> 4
- net SCL: track 68.2 -> 68.7 mm

Commit message: Post-review updates
Parts:
- removed D3: 1A/23V/620mV, SparkFun-DiscreteSemi:SOD-323
- removed L1: 15uH, SparkFun-Coils:INDUCTOR_LQH32
- added R4: 4.7k, SparkFun-Resistors:0402-TIGHT
- added RXD0, TXD0: TEST-POINT3X4, SparkFun-Connectors:PAD.03X.04
- added U5: ATTINY841-ARDUINO_QFN20M1, SparkFun-IC-Microcontroller:QFN20_20M1
- C5: value 4.7uF -> 2.2uF
- C7: value 22uF -> 2.2uF; device SparkFun-Capacitors:0603 -> SparkFun-Capacitors:0402-TIGHT
- U1: value ATTINY43_QFN20 -> STLQ015-3.3V; device New-Parts_SparkFun-IC-Microcontroller:QFN20_20M1 -> SparkFun-IC-Power:SOT23-5
- moved U$1 12.1 mm to (1.21, 11.9), turned to 90 degrees
- moved U$5 10.2 mm to (2.92, 29.2)
- moved VIN 10.2 mm to (5.08, 29.2)
- moved C8 8.21 mm to (8.89, 20.4), turned to 0 degrees
- moved U$2 7.73 mm to (0.76, 20.1), turned to 90 degrees
- moved C7 5.15 mm to (4.54, 15.3), turned to 180 degrees
- moved U1 4.47 mm to (7.87, 15.4), turned to 90 degrees
- moved U$20 3.81 mm to (5.33, 25.4)
- moved U$3 3.30 mm to (5.33, 23.4)
- moved LOGO3 2.54 mm to (5.33, 21.0)
- moved LOGO2 1.23 mm to (1.46, 6.79), turned to 90 degrees
- moved C5 0.91 mm to (9.65, 17.8), turned to 90 degrees
Connections:
- removed net N$2: D3.A, L1.P$1, U1.9
- new net RXD0: RXD0.1, U5.3
- new net TXD0: TXD0.1, U5.4
- net !RESET!: now also R4.1, U5.13; no longer U1.18
- net 3V3_EN: now also U5.5; no longer U1.14
- net AT_CIPO: now also U5.20; no longer U1.4
- net AT_VCC: now also R4.2, U1.5, U5.9; no longer D3.C, U1.7
- net GND: now also U1.2, U5.8, U5.PAD; no longer U1.8, U1.PAD
- net SCL: now also U5.1; no longer U1.5
- net SDA: now also U5.16; no longer U1.3
- net VIN: now also U1.1, U1.3; no longer L1.P$2, U1.10
Routing:
- net GND: track 89.4 -> 57.4 mm, vias 46 -> 44
- net AT_CIPO: track 20.7 -> 15.2 mm
- net RXD0: track 0.00 -> 4.39 mm, vias 0 -> 1
- net N$2: track 3.40 -> 0.00 mm
- net AT_VCC: track 14.8 -> 17.7 mm, vias 0 -> 2
- net TXD0: track 0.00 -> 2.89 mm, vias 0 -> 1
- net 3V3_EN: track 30.7 -> 32.9 mm
- net SDA: track 60.8 -> 59.2 mm
- net !RESET!: track 18.3 -> 19.6 mm
- net SCL: track 68.7 -> 69.5 mm
- net 3.3V: track 77.3 -> 76.5 mm

Commit message: Post-review updates
Parts:
- added U$10: (no value), output:CHG0
- added U$11: (no value), output:5#5V_MAX0
- added U$14: (no value), output:#RXD0#0
- added U$15: (no value), output:#TXD0#0
- moved U$2 10.9 mm to (9.65, 26.5)
- moved FG_SDA 2.18 mm to (8.06, 28.9), flipped to the bottom
- moved U$9 1.35 mm to (9.81, 28.7), flipped to the bottom
- moved U$1 0.92 mm to (1.46, 12.8)
- moved U5 0.25 mm to (5.33, 19.3)
- moved LOGO2 0.20 mm to (1.52, 6.99)
Routing:
- net GND: track 57.4 -> 82.0 mm, vias 44 -> 47
- net N$1: track 6.97 -> 2.94 mm, vias 2 -> 1
- net SDA: track 59.2 -> 61.3 mm, vias 5 -> 6

Commit message: Final tweaks
Parts:
- added U$16: (no value), output:5#5V0
- U$11: device output:5#5V_MAX0 -> output:MAX0
- moved U$10 3.81 mm to (0.57, 22.7)
- moved U$11 3.54 mm to (9.21, 31.0), turned to 0 degrees
- moved U$2 0.46 mm to (9.78, 26.0)
- moved R1 0.32 mm to (2.48, 22.7)
- moved RPROG 0.32 mm to (2.48, 23.7)
Routing:
- net GND: track 82.0 -> 96.0 mm

Commit message: Gapless production panel
Other:
- board text added: "2-Layer Board 1.6mm Thickness 1oz Copper (Outer layers) HASL Finish"
- board text removed: "2-Layer Board 1.6mm Thickness 1oz Copper (Outer layers) HASL Finish When running the panelizer, add a vertical gap of 0.2" to make the boards easier to separate"
Changed lines of the file:
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@@
 <setting verticaltext="up"/>
 </settings>
-<grid distance="0.05" unitdist="inch" unit="inch" style="lines" multiple="1" display="yes" altdistance="0.00125" altunitdist="inch" altunit="inch"/>
+<grid distance="0.05" unitdist="inch" unit="inch" style="lines" multiple="1" display="yes" altdistance="0.0025" altunitdist="inch" altunit="inch"/>
 <layers>
 <layer number="1" name="Top" color="4" fill="1" visible="yes" active="yes"/>
@@
 <layer number="23" name="tOrigins" color="15" fill="1" visible="yes" active="yes"/>
 <layer number="24" name="bOrigins" color="15" fill="1" visible="yes" active="yes"/>
-<layer number="25" name="tNames" color="57" fill="1" visible="yes" active="yes"/>
-<layer number="26" name="bNames" color="57" fill="1" visible="yes" active="yes"/>
-<layer number="27" name="tValues" color="7" fill="1" visible="yes" active="yes"/>
-<layer number="28" name="bValues" color="7" fill="1" visible="yes" active="yes"/>
-<layer number="29" name="tStop" color="7" fill="3" visible="yes" active="yes"/>
-<layer number="30" name="bStop" color="7" fill="6" visible="yes" active="yes"/>
-<layer number="31" name="tCream" color="7" fill="4" visible="yes" active="yes"/>
-<layer number="32" name="bCream" color="7" fill="5" visible="yes" active="yes"/>
-<layer number="33" name="tFinish" color="6" fill="3" visible="yes" active="yes"/>
-<layer number="34" name="bFinish" color="6" fill="6" visible="yes" active="yes"/>
-<layer number="35" name="tGlue" color="7" fill="4" visible="yes" active="yes"/>
-<layer number="36" name="bGlue" color="7" fill="5" visible="yes" active="yes"/>
-<layer number="37" name="tTest" color="7" fill="1" visible="yes" active="yes"/>
-<layer number="38" name="bTest" color="7" fill="1" visible="yes" active="yes"/>
-<layer number="39" name="tKeepout" color="4" fill="11" visible="yes" active="yes"/>
-<layer number="40" name="bKeepout" color="1" fill="11" visible="yes" active="yes"/>
-<layer number="41" name="tRestrict" color="4" fill="10" visible="yes" active="yes"/>
-<layer number="42" name="bRestrict" color="1" fill="10" visible="yes" active="yes"/>
-<layer number="43" name="vRestrict" color="2" fill="10" visible="yes" active="yes"/>
-<layer number="44" name="Drills" color="7" fill="1" visible="yes" active="yes"/>
+<layer number="25" name="tNames" color="57" fill="1" visible="no" active="yes"/>
+<layer number="26" name="bNames" color="57" fill="1" visible="no" active="yes"/>
+<layer number="27" name="tValues" color="7" fill="1" visible="no" active="yes"/>
+<layer number="28" name="bValues" color="7" fill="1" visible="no" active="yes"/>
+<layer number="29" name="tStop" color="7" fill="3" visible="no" active="yes"/>
+<layer number="30" name="bStop" color="7" fill="6" visible="no" active="yes"/>
+<layer number="31" name="tCream" color="7" fill="4" visible="no" active="yes"/>
+<layer number="32" name="bCream" color="7" fill="5" visible="no" active="yes"/>
+<layer number="33" name="tFinish" color="6" fill="3" visible="no" active="yes"/>
+<layer number="34" name="bFinish" color="6" fill="6" visible="no" active="yes"/>
+<layer number="35" name="tGlue" color="7" fill="4" visible="no" active="yes"/>
+<layer number="36" name="bGlue" color="7" fill="5" visible="no" active="yes"/>
+<layer number="37" name="tTest" color="7" fill="1" visible="no" active="yes"/>
+<layer number="38" name="bTest" color="7" fill="1" visible="no" active="yes"/>
+<layer number="39" name="tKeepout" color="4" fill="11" visible="no" active="yes"/>
+<layer number="40" name="bKeepout" color="1" fill="11" visible="no" active="yes"/>
+<layer number="41" name="tRestrict" color="4" fill="10" visible="no" active="yes"/>
+<layer number="42" name="bRestrict" color="1" fill="10" visible="no" active="yes"/>
+<layer number="43" name="vRestrict" color="2" fill="10" visible="no" active="yes"/>
+<layer number="44" name="Drills" color="7" fill="1" visible="no" active="yes"/>
 <layer number="45" name="Holes" color="7" fill="1" visible="yes" active="yes"/>
-<layer number="46" name="Milling" color="3" fill="1" visible="yes" active="yes"/>
-<layer number="47" name="Measures" color="7" fill="1" visible="yes" active="yes"/>
-<layer number="48" name="Document" color="7" fill="1" visible="yes" active="yes"/>
-<layer number="49" name="Reference" color="7" fill="1" visible="yes" active="yes"/>
-<layer number="50" name="dxf" color="7" fill="1" visible="yes" active="yes"/>
+<layer number="46" name="Milling" color="3" fill="1" visible="no" active="yes"/>
+<layer number="47" name="Measures" color="7" fill="1" visible="no" active="yes"/>
+<layer number="48" name="Document" color="7" fill="1" visible="no" active="yes"/>
+<layer number="49" name="Reference" color="7" fill="1" visible="no" active="yes"/>
+<layer number="50" name="dxf" color="7" fill="1" visible="no" active="yes"/>
 <layer number="51" name="tDocu" color="6" fill="1" visible="yes" active="yes"/>
-<layer number="52" name="bDocu" color="7" fill="1" visible="yes" active="yes"/>
+<layer number="52" name="bDocu" color="7" fill="1" visible="no" active="yes"/>
 <layer number="2" name="Route2" color="63" fill="1" visible="no" active="no"/>
 <layer number="15" name="Route15" color="23" fill="1" visible="no" active="no"/>
@@
 1oz Copper (Outer layers)
 HASL Finish
-When running the panelizer, add a vertical gap of 0.2"
-to make the boards easier to separate</text>
+</text>
 <dimension x1="0" y1="0" x2="10.668" y2="0" x3="5.334" y3="-3.81" textsize="1.778" textratio="15" layer="47" dtype="horizontal" unit="inch"/>
 <dimension x1="0" y1="40.64" x2="0" y2="0" x3="-3.810003125" y3="20.32" textsize="1.778" textratio="15" layer="47" dtype="vertical" unit="inch"/>

Commit message: Update 16-way FPC Connector. Add missing PROD_IDs
Parts:
- IN, OUT: value FPC_16_0.5MM_BACKFLIP -> (none); device New_Parts_Connectors:FPC_16_DOUBLESIDED_BACKFLIP -> SparkFun-Connectors:FPC_16_0.5MM
Changed lines of the file:
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@@
 <element name="FD3" library="SparkFun-Aesthetics" package="FIDUCIAL-MICRO" value="FIDUCIALUFIDUCIAL" x="10.033" y="0.635" smashed="yes"/>
 <element name="FD4" library="SparkFun-Aesthetics" package="FIDUCIAL-MICRO" value="FIDUCIALUFIDUCIAL" x="10.033" y="0.635" smashed="yes" rot="MR0"/>
-<element name="OUT" library="New_Parts_Connectors" package="FPC_16_DOUBLESIDED_BACKFLIP" value="FPC_16_0.5MM_BACKFLIP" x="5.334" y="2.0955" smashed="yes" rot="R180">
-<attribute name="ATOM_PART" value="FPC05016-42201" x="5.334" y="2.0955" size="1.778" layer="27" font="vector" ratio="15" rot="R180" display="off"/>
-<attribute name="PROD_ID" value="" x="5.334" y="2.0955" size="1.778" layer="27" font="vector" ratio="15" rot="R180" display="off"/>
+<element name="OUT" library="SparkFun-Connectors" package="FPC_16_0.5MM" value="" x="5.334" y="2.0955" smashed="yes" rot="R180">
+<attribute name="PROD_ID" value="CONN-16066" x="5.334" y="2.0955" size="1.778" layer="27" font="vector" ratio="15" rot="R180" display="off"/>
 </element>
 <element name="LOGO2" library="SparkFun-Aesthetics" package="OSHW-LOGO-MINI" value="OSHW-LOGOMINI" x="1.524" y="6.985" smashed="yes" rot="R90"/>
@@
 <element name="U$20" library="SparkX" package="SPARKX-SMALL" value="SPARKX-LOGO3" x="5.334" y="25.4" smashed="yes" rot="MR0"/>
 <element name="LOGO3" library="SparkFun-Aesthetics" package="OSHW-LOGO-MINI" value="OSHW-LOGOMINI" x="5.334" y="20.955" smashed="yes" rot="MR0"/>
-<element name="IN" library="New_Parts_Connectors" package="FPC_16_DOUBLESIDED_BACKFLIP" value="FPC_16_0.5MM_BACKFLIP" x="5.334" y="38.5445" smashed="yes" rot="MR0">
-<attribute name="ATOM_PART" value="FPC05016-42201" x="5.334" y="38.5445" size="1.778" layer="28" ratio="15" rot="MR0" display="off"/>
-<attribute name="PROD_ID" value="" x="5.334" y="38.5445" size="1.778" layer="28" ratio="15" rot="MR0" display="off"/>
+<element name="IN" library="SparkFun-Connectors" package="FPC_16_0.5MM" value="" x="5.334" y="38.5445" smashed="yes" rot="MR0">
+<attribute name="PROD_ID" value="CONN-16066" x="5.334" y="38.5445" size="1.778" layer="28" ratio="15" rot="MR0" display="off"/>
 </element>
 <element name="U$12" library="output" package="#IN#0" value="" x="5.334" y="34.798" smashed="yes" rot="MR0"/>
@@
 <attribute name="DIGIKEY_PART" value="ATTINY841-MU-ND" x="5.334" y="19.304" size="1.778" layer="27" ratio="15" rot="R90" display="off"/>
 <attribute name="NAME" x="2.842" y="17.939" size="0.6096" layer="25" ratio="20" rot="R90"/>
-<attribute name="PROD_ID" value="" x="5.334" y="19.304" size="1.778" layer="27" ratio="15" rot="R90" display="off"/>
+<attribute name="PROD_ID" value="IC-16067" x="5.334" y="19.304" size="1.778" layer="27" ratio="15" rot="R90" display="off"/>
 </element>
 <element name="R4" library="SparkFun-Resistors" package="0402-TIGHT" value="4.7k" x="8.9535" y="21.5265" smashed="yes">
