File: Hardware/SparkX_EZ_LiPo_Power.sch (EAGLE design)
At the start: 39 parts, among them J3 AVR_SPI_PROG_3X2TESTPOINTS, Q1 3.1A/30V/105mΩ, U1 ATTINY43_QFN20, U2 MCP73831, U3 3.3V, U4 MAX17048

Commit message: Partially routed
Parts:
- removed J2: (no value), SparkFun-Connectors:CONN_021X02_NO_SILK
- added BATT+: TEST-POINT3X4, SparkFun-Connectors:TEST-POINT3X4
- added FG_SDA: JUMPER-SMT_2_NC_TRACE_SILK, SparkFun-Jumpers:JUMPER-SMT_2_NC_TRACE_SILK
Connections:
- new net N$1: FG_SDA.1, U4.SDA
- net GND: no longer J2.2
- net SDA: now also FG_SDA.2; no longer U4.SDA
- net V_BATT: now also BATT+.1; no longer J2.1
Other:
- moved on the sheet: J1
Changed lines of the file:
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@@
 <part name="SUPPLY7" library="SparkFun-PowerSymbols" deviceset="V_BATT" device=""/>
 <part name="J1" library="SparkFun-Connectors" deviceset="JST_2MM_MALE" device=""/>
-<part name="J2" library="SparkFun-Connectors" deviceset="CONN_02" device="1X02_NO_SILK"/>
 <part name="GND35" library="SparkFun-PowerSymbols" deviceset="GND" device=""/>
 <part name="SUPPLY1" library="SparkFun-PowerSymbols" deviceset="V_USB" device=""/>
@@
 <part name="GND11" library="SparkFun-PowerSymbols" deviceset="GND" device=""/>
 <part name="AT_VCC" library="SparkFun-Jumpers" deviceset="JUMPER-SMT_2_NC_TRACE" device="_SILK" package3d_urn="urn:adsk.eagle:package:39281/1"/>
+<part name="FG_SDA" library="SparkFun-Jumpers" deviceset="JUMPER-SMT_2_NC_TRACE" device="_SILK" package3d_urn="urn:adsk.eagle:package:39281/1"/>
+<part name="BATT+" library="SparkFun-Connectors" deviceset="TEST-POINT" device="3X4" value="TEST-POINT3X4"/>
 </parts>
 <sheets>
@@
 <attribute name="VALUE" x="208.28" y="251.714" size="1.778" layer="96" font="vector" align="bottom-center"/>
 </instance>
-<instance part="J1" gate="G$1" x="241.3" y="243.84" smashed="yes" rot="MR90">
-<attribute name="NAME" x="245.11" y="240.538" size="1.778" layer="95" font="vector" rot="MR180"/>
-</instance>
-<instance part="J2" gate="G$1" x="243.84" y="231.14" smashed="yes" rot="R180">
-<attribute name="VALUE" x="246.38" y="235.966" size="1.778" layer="96" font="vector" rot="R180"/>
-<attribute name="NAME" x="246.38" y="225.552" size="1.778" layer="95" font="vector" rot="R180"/>
+<instance part="J1" gate="G$1" x="241.3" y="236.22" smashed="yes" rot="MR90">
+<attribute name="NAME" x="245.11" y="232.918" size="1.778" layer="95" font="vector" rot="MR180"/>
 </instance>
 <instance part="GND35" gate="1" x="208.28" y="223.52" smashed="yes">
@@
 <instance part="AT_VCC" gate="G$1" x="220.98" y="142.24" smashed="yes">
 <attribute name="NAME" x="215.9" y="144.78" size="1.778" layer="95" font="vector"/>
+</instance>
+<instance part="FG_SDA" gate="G$1" x="414.02" y="241.3" smashed="yes">
+<attribute name="NAME" x="408.94" y="243.84" size="1.778" layer="95" font="vector"/>
+</instance>
+<instance part="BATT+" gate="G$1" x="236.22" y="246.38" smashed="yes">
+<attribute name="NAME" x="236.22" y="248.92" size="1.778" layer="95" font="vector"/>
 </instance>
 </instances>
@@
 <junction x="213.36" y="228.6"/>
 <wire x1="220.98" y1="228.6" x2="213.36" y2="228.6" width="0.1524" layer="91"/>
-<wire x1="236.22" y1="243.84" x2="233.68" y2="243.84" width="0.1524" layer="91"/>
-<wire x1="233.68" y1="243.84" x2="233.68" y2="228.6" width="0.1524" layer="91"/>
+<wire x1="236.22" y1="236.22" x2="233.68" y2="236.22" width="0.1524" layer="91"/>
+<wire x1="233.68" y1="236.22" x2="233.68" y2="228.6" width="0.1524" layer="91"/>
 <wire x1="233.68" y1="228.6" x2="220.98" y2="228.6" width="0.1524" layer="91"/>
 <junction x="220.98" y="228.6"/>
 <pinref part="J1" gate="G$1" pin="-"/>
-<pinref part="J2" gate="G$1" pin="2"/>
-<wire x1="236.22" y1="228.6" x2="233.68" y2="228.6" width="0.1524" layer="91"/>
-<junction x="233.68" y="228.6"/>
 <pinref part="GND35" gate="1" pin="GND"/>
 </segment>
@@
 </segment>
 <segment>
-<pinref part="U4" gate="U1" pin="SDA"/>
-<wire x1="406.4" y1="241.3" x2="408.94" y2="241.3" width="0.1524" layer="91"/>
-<label x="408.94" y="241.3" size="1.27" layer="95" xref="yes"/>
+<label x="421.64" y="241.3" size="1.27" layer="95" xref="yes"/>
+<pinref part="FG_SDA" gate="G$1" pin="2"/>
+<wire x1="419.1" y1="241.3" x2="421.64" y2="241.3" width="0.1524" layer="91"/>
 </segment>
 <segment>
 <pinref part="U1" gate="G$1" pin="D4/DI/COPI/SDA"/>
-<wire x1="185.42" y1="99.06" x2="175.26" y2="99.06" width="0.1524" layer="91"/>
-<label x="175.26" y="99.06" size="1.27" layer="95" rot="R180" xref="yes"/>
+<wire x1="185.42" y1="101.6" x2="182.88" y2="101.6" width="0.1524" layer="91"/>
+<label x="182.88" y="101.6" size="1.27" layer="95" rot="R180" xref="yes"/>
 </segment>
 <segment>
@@
 <segment>
 <pinref part="U1" gate="G$1" pin="D6/SCK/SCL"/>
-<wire x1="185.42" y1="93.98" x2="175.26" y2="93.98" width="0.1524" layer="91"/>
-<label x="175.26" y="93.98" size="1.27" layer="95" font="vector" rot="R180" xref="yes"/>
+<wire x1="185.42" y1="96.52" x2="182.88" y2="96.52" width="0.1524" layer="91"/>
+<label x="182.88" y="96.52" size="1.27" layer="95" font="vector" rot="R180" xref="yes"/>
 </segment>
 <segment>
@@
 <pinref part="U2" gate="G$1" pin="VBAT"/>
 <pinref part="C6" gate="G$1" pin="1"/>
-<wire x1="236.22" y1="246.38" x2="231.14" y2="246.38" width="0.1524" layer="91"/>
-<wire x1="231.14" y1="246.38" x2="220.98" y2="246.38" width="0.1524" layer="91"/>
+<wire x1="236.22" y1="238.76" x2="233.68" y2="238.76" width="0.1524" layer="91"/>
+<wire x1="233.68" y1="238.76" x2="233.68" y2="246.38" width="0.1524" layer="91"/>
+<wire x1="233.68" y1="246.38" x2="220.98" y2="246.38" width="0.1524" layer="91"/>
 <wire x1="220.98" y1="246.38" x2="208.28" y2="246.38" width="0.1524" layer="91"/>
 <wire x1="208.28" y1="246.38" x2="205.74" y2="246.38" width="0.1524" layer="91"/>
@@
 <junction x="220.98" y="246.38"/>
 <pinref part="J1" gate="G$1" pin="+"/>
-<pinref part="J2" gate="G$1" pin="1"/>
-<wire x1="236.22" y1="231.14" x2="231.14" y2="231.14" width="0.1524" layer="91"/>
-<wire x1="231.14" y1="231.14" x2="231.14" y2="246.38" width="0.1524" layer="91"/>
-<junction x="231.14" y="246.38"/>
 <pinref part="SUPPLY7" gate="G$1" pin="V_BATT"/>
 <wire x1="208.28" y1="248.92" x2="208.28" y2="246.38" width="0.1524" layer="91"/>
 <junction x="208.28" y="246.38"/>
+<pinref part="BATT+" gate="G$1" pin="1"/>
+<wire x1="236.22" y1="246.38" x2="233.68" y2="246.38" width="0.1524" layer="91"/>
+<junction x="233.68" y="246.38"/>
 </segment>
 <segment>
@@
 <segment>
 <pinref part="U1" gate="G$1" pin="VCC"/>
-<wire x1="185.42" y1="111.76" x2="177.8" y2="111.76" width="0.1524" layer="91"/>
+<wire x1="185.42" y1="91.44" x2="177.8" y2="91.44" width="0.1524" layer="91"/>
 <pinref part="C7" gate="G$1" pin="1"/>
-<wire x1="177.8" y1="111.76" x2="177.8" y2="76.2" width="0.1524" layer="91"/>
+<wire x1="177.8" y1="91.44" x2="177.8" y2="76.2" width="0.1524" layer="91"/>
 <pinref part="D3" gate="G$1" pin="C"/>
 <wire x1="177.8" y1="76.2" x2="177.8" y2="73.66" width="0.1524" layer="91"/>
@@
 <wire x1="187.96" y1="73.66" x2="187.96" y2="76.2" width="0.1524" layer="91"/>
 <junction x="187.96" y="76.2"/>
-<wire x1="177.8" y1="111.76" x2="175.26" y2="111.76" width="0.1524" layer="91"/>
-<junction x="177.8" y="111.76"/>
-<label x="175.26" y="111.76" size="1.27" layer="95" font="vector" rot="R180" xref="yes"/>
+<wire x1="177.8" y1="91.44" x2="175.26" y2="91.44" width="0.1524" layer="91"/>
+<junction x="177.8" y="91.44"/>
+<label x="175.26" y="91.44" size="1.27" layer="95" font="vector" rot="R180" xref="yes"/>
 </segment>
 <segment>
@@
 <segment>
 <pinref part="U1" gate="G$1" pin="D5/DO/CIPO"/>
-<wire x1="185.42" y1="96.52" x2="175.26" y2="96.52" width="0.1524" layer="91"/>
-<label x="175.26" y="96.52" size="1.27" layer="95" font="vector" rot="R180" xref="yes"/>
+<wire x1="185.42" y1="99.06" x2="182.88" y2="99.06" width="0.1524" layer="91"/>
+<label x="182.88" y="99.06" size="1.27" layer="95" font="vector" rot="R180" xref="yes"/>
 </segment>
 <segment>
@@
 </segment>
 </net>
+<net name="N$1" class="0">
+<segment>
+<pinref part="U4" gate="U1" pin="SDA"/>
+<pinref part="FG_SDA" gate="G$1" pin="1"/>
+<wire x1="406.4" y1="241.3" x2="408.94" y2="241.3" width="0.1524" layer="91"/>
+</segment>
+</net>

Commit message: Freshly routed
Other:
- moved on the sheet: AT_VCC, C5, C7, C8, D3, J3, L1, U1

Commit message: Post-review updates
Parts:
- removed D3: 1A/23V/620mV, SparkFun-DiscreteSemi:DIODE-SCHOTTKY-BAT20J
- removed L1: 15uH, SparkFun-Coils:INDUCTOR-LHQ32-15UH
- added R4: 4.7k, SparkFun-Resistors:4.7KOHM-0402T-1/16W-1%
- added RXD0, TXD0: TEST-POINT3X4, SparkFun-Connectors:TEST-POINT3X4
- added U5: ATTINY841-ARDUINO_QFN20M1, SparkFun-IC-Microcontroller:ATTINY841-ARDUINO_QFN20M1
- C5: value 4.7uF -> 2.2uF; device SparkFun-Capacitors:4.7UF-0402_TIGHT-6.3V-20%-X5R -> SparkFun-Capacitors:2.2UF-0402_TIGHT-10V-10%-X5R
- C7: value 22uF -> 2.2uF; device SparkFun-Capacitors:22UF-0603-6.3V-20% -> SparkFun-Capacitors:2.2UF-0402_TIGHT-10V-10%-X5R
- U1: value ATTINY43_QFN20 -> STLQ015-3.3V; device New-Parts_SparkFun-IC-Microcontroller:ATTINY43_QFN20 -> SparkFun-IC-Power:STLQ015-3.3V
Connections:
- removed net N$2: D3.A, L1.1, U1.LSW
- new net RXD0: RXD0.1, U5.(RXD0/A2)2
- new net TXD0: TXD0.1, U5.(TXD0/A1)1
- net !RESET!: now also R4.1, U5.(!RESET!/A9)11; no longer U1.!RESET!/D15
- net 3V3_EN: now also U5.(A0)0; no longer U1.A3/D11
- net AT_CIPO: now also U5.(CIPO/A5)5; no longer U1.D5/DO/CIPO
- net AT_VCC: now also R4.2, U1.OUT, U5.VCC; no longer D3.C, U1.VCC
- net GND: now also U5.GND
- net SCL: now also U5.(SCL/SCK/A4)4; no longer U1.D6/SCK/SCL
- net SDA: now also U5.(SDA/COPI/A6)6; no longer U1.D4/DI/COPI/SDA
- net VIN: now also U1.EN, U1.IN; no longer L1.2, U1.VBAT
Other:
- note added: "ATtiny Voltage Regulation"
- note added: "EZ Voltage Regulation"
- note added: "STLQ015-3.3V ---------- Iout (max): 150mA Vin (max): 5.5V Vdrop (typ): 112mV Iq: 1.4uA"
- note removed: "ATtiny43 ====== Pin 4 is COPI and Pin 5 is CIPO when the chip is in peripheral mode or is being programmed Pin 4 is CIPO and Pin 5 is COPI when the chip is operating in controller mode The #defines in the ATTinyCore assume controller mode"
- note removed: "Voltage Regulation"
- moved on the sheet: AT_VCC, C5, C7, C8, J3

Commit message: Post-review updates
Other:
- note added: "ATtiny841"
- note removed: "ATtiny43"
- moved on the sheet: C4, FG_SDA, U4
Changed lines of the file:
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@@
 <text x="357.124" y="268.732" size="5.08" layer="94">Fuel Gauge</text>
 <wire x1="431.8" y1="190.5" x2="350.52" y2="190.5" width="0.2032" layer="97" style="longdash"/>
-<text x="390.779" y="212.471" size="2.54" layer="97" font="vector" align="center">I2C Address = 0x36</text>
-<text x="6.604" y="179.832" size="5.08" layer="94">ATtiny43</text>
+<text x="385.699" y="209.931" size="2.54" layer="97" font="vector" align="center">I2C Address = 0x36</text>
+<text x="6.604" y="179.832" size="5.08" layer="94">ATtiny841</text>
 <wire x1="154.94" y1="0" x2="154.94" y2="101.6" width="0.2032" layer="97" style="longdash"/>
 <text x="200.66" y="129.54" size="1.27" layer="97" align="top-left">STLQ015-3.3V
@@
 <attribute name="VALUE" x="332.74" y="223.774" size="1.778" layer="96" align="bottom-center"/>
 </instance>
-<instance part="U4" gate="U1" x="396.24" y="238.76" smashed="yes">
-<attribute name="NAME" x="386.08" y="249.428" size="1.778" layer="95" font="vector"/>
-<attribute name="VALUE" x="386.08" y="226.06" size="1.778" layer="96" font="vector"/>
-</instance>
-<instance part="SUPPLY3" gate="G$1" x="381" y="248.92" smashed="yes" rot="MR0">
-<attribute name="VALUE" x="381" y="251.714" size="1.778" layer="96" font="vector" rot="MR0" align="bottom-center"/>
-</instance>
-<instance part="GND43" gate="1" x="381" y="226.06" smashed="yes">
-<attribute name="VALUE" x="381" y="225.806" size="1.778" layer="96" align="top-center"/>
-</instance>
-<instance part="GND76" gate="1" x="408.94" y="226.06" smashed="yes">
-<attribute name="VALUE" x="408.94" y="225.806" size="1.778" layer="96" align="top-center"/>
+<instance part="U4" gate="U1" x="391.16" y="236.22" smashed="yes">
+<attribute name="NAME" x="381" y="246.888" size="1.778" layer="95" font="vector"/>
+<attribute name="VALUE" x="381" y="223.52" size="1.778" layer="96" font="vector"/>
+</instance>
+<instance part="SUPPLY3" gate="G$1" x="375.92" y="246.38" smashed="yes" rot="MR0">
+<attribute name="VALUE" x="375.92" y="249.174" size="1.778" layer="96" font="vector" rot="MR0" align="bottom-center"/>
+</instance>
+<instance part="GND43" gate="1" x="375.92" y="223.52" smashed="yes">
+<attribute name="VALUE" x="375.92" y="223.266" size="1.778" layer="96" align="top-center"/>
+</instance>
+<instance part="GND76" gate="1" x="403.86" y="223.52" smashed="yes">
+<attribute name="VALUE" x="403.86" y="223.266" size="1.778" layer="96" align="top-center"/>
 </instance>
 <instance part="D2" gate="G$1" x="289.56" y="241.3" smashed="yes">
@@
 <attribute name="VALUE" x="279.4" y="218.694" size="1.778" layer="96" align="bottom-center"/>
 </instance>
-<instance part="C4" gate="G$1" x="370.84" y="238.76" smashed="yes">
-<attribute name="NAME" x="372.364" y="241.681" size="1.778" layer="95" font="vector"/>
-<attribute name="VALUE" x="372.364" y="236.601" size="1.778" layer="96" font="vector"/>
-</instance>
-<instance part="GND6" gate="1" x="370.84" y="231.14" smashed="yes">
-<attribute name="VALUE" x="370.84" y="230.886" size="1.778" layer="96" font="vector" align="top-center"/>
-</instance>
-<instance part="SUPPLY10" gate="G$1" x="370.84" y="246.38" smashed="yes" rot="MR0">
-<attribute name="VALUE" x="370.84" y="249.174" size="1.778" layer="96" font="vector" rot="MR0" align="bottom-center"/>
+<instance part="C4" gate="G$1" x="365.76" y="236.22" smashed="yes">
+<attribute name="NAME" x="367.284" y="239.141" size="1.778" layer="95" font="vector"/>
+<attribute name="VALUE" x="367.284" y="234.061" size="1.778" layer="96" font="vector"/>
+</instance>
+<instance part="GND6" gate="1" x="365.76" y="228.6" smashed="yes">
+<attribute name="VALUE" x="365.76" y="228.346" size="1.778" layer="96" font="vector" align="top-center"/>
+</instance>
+<instance part="SUPPLY10" gate="G$1" x="365.76" y="243.84" smashed="yes" rot="MR0">
+<attribute name="VALUE" x="365.76" y="246.634" size="1.778" layer="96" font="vector" rot="MR0" align="bottom-center"/>
 </instance>
 <instance part="VIN" gate="G$1" x="304.8" y="241.3" smashed="yes">
@@
 <attribute name="NAME" x="88.9" y="129.54" size="1.778" layer="95" font="vector"/>
 </instance>
-<instance part="FG_SDA" gate="G$1" x="414.02" y="241.3" smashed="yes">
-<attribute name="NAME" x="408.94" y="243.84" size="1.778" layer="95" font="vector"/>
+<instance part="FG_SDA" gate="G$1" x="408.94" y="238.76" smashed="yes">
+<attribute name="NAME" x="403.86" y="241.3" size="1.778" layer="95" font="vector"/>
 </instance>
 <instance part="BATT+" gate="G$1" x="236.22" y="246.38" smashed="yes">
@@
 <segment>
 <pinref part="U4" gate="U1" pin="GND"/>
-<wire x1="383.54" y1="231.14" x2="381" y2="231.14" width="0.1524" layer="91"/>
+<wire x1="378.46" y1="228.6" x2="375.92" y2="228.6" width="0.1524" layer="91"/>
 <pinref part="GND43" gate="1" pin="GND"/>
-<wire x1="381" y1="231.14" x2="381" y2="228.6" width="0.1524" layer="91"/>
+<wire x1="375.92" y1="228.6" x2="375.92" y2="226.06" width="0.1524" layer="91"/>
 <pinref part="U4" gate="U1" pin="CTG"/>
-<wire x1="383.54" y1="236.22" x2="381" y2="236.22" width="0.1524" layer="91"/>
-<wire x1="381" y1="236.22" x2="381" y2="231.14" width="0.1524" layer="91"/>
-<junction x="381" y="231.14"/>
+<wire x1="378.46" y1="233.68" x2="375.92" y2="233.68" width="0.1524" layer="91"/>
+<wire x1="375.92" y1="233.68" x2="375.92" y2="228.6" width="0.1524" layer="91"/>
+<junction x="375.92" y="228.6"/>
 </segment>
 <segment>
 <pinref part="U4" gate="U1" pin="QSTRT"/>
-<wire x1="406.4" y1="231.14" x2="408.94" y2="231.14" width="0.1524" layer="91"/>
+<wire x1="401.32" y1="228.6" x2="403.86" y2="228.6" width="0.1524" layer="91"/>
 <pinref part="GND76" gate="1" pin="GND"/>
-<wire x1="408.94" y1="231.14" x2="408.94" y2="228.6" width="0.1524" layer="91"/>
+<wire x1="403.86" y1="228.6" x2="403.86" y2="226.06" width="0.1524" layer="91"/>
 </segment>
 <segment>
@@
 <pinref part="C4" gate="G$1" pin="2"/>
 <pinref part="GND6" gate="1" pin="GND"/>
-<wire x1="370.84" y1="236.22" x2="370.84" y2="233.68" width="0.1524" layer="91"/>
+<wire x1="365.76" y1="233.68" x2="365.76" y2="231.14" width="0.1524" layer="91"/>
 </segment>
 <segment>
@@
 </segment>
 <segment>
-<label x="421.64" y="241.3" size="1.27" layer="95" xref="yes"/>
+<label x="416.56" y="238.76" size="1.27" layer="95" xref="yes"/>
 <pinref part="FG_SDA" gate="G$1" pin="2"/>
-<wire x1="419.1" y1="241.3" x2="421.64" y2="241.3" width="0.1524" layer="91"/>
+<wire x1="414.02" y1="238.76" x2="416.56" y2="238.76" width="0.1524" layer="91"/>
 </segment>
 <segment>
@@
 <segment>
 <pinref part="U4" gate="U1" pin="SCL"/>
-<wire x1="406.4" y1="236.22" x2="408.94" y2="236.22" width="0.1524" layer="91"/>
-<label x="408.94" y="236.22" size="1.27" layer="95" xref="yes"/>
+<wire x1="401.32" y1="233.68" x2="403.86" y2="233.68" width="0.1524" layer="91"/>
+<label x="403.86" y="233.68" size="1.27" layer="95" xref="yes"/>
 </segment>
 <segment>
@@
 <segment>
 <pinref part="U4" gate="U1" pin="CELL"/>
-<wire x1="383.54" y1="241.3" x2="381" y2="241.3" width="0.1524" layer="91"/>
+<wire x1="378.46" y1="238.76" x2="375.92" y2="238.76" width="0.1524" layer="91"/>
 <pinref part="SUPPLY3" gate="G$1" pin="V_BATT"/>
-<wire x1="381" y1="241.3" x2="381" y2="246.38" width="0.1524" layer="91"/>
+<wire x1="375.92" y1="238.76" x2="375.92" y2="243.84" width="0.1524" layer="91"/>
 <pinref part="U4" gate="U1" pin="VDD"/>
-<wire x1="381" y1="246.38" x2="381" y2="248.92" width="0.1524" layer="91"/>
-<wire x1="383.54" y1="246.38" x2="381" y2="246.38" width="0.1524" layer="91"/>
-<junction x="381" y="246.38"/>
+<wire x1="375.92" y1="243.84" x2="375.92" y2="246.38" width="0.1524" layer="91"/>
+<wire x1="378.46" y1="243.84" x2="375.92" y2="243.84" width="0.1524" layer="91"/>
+<junction x="375.92" y="243.84"/>
 </segment>
 <segment>
@@
 <pinref part="SUPPLY10" gate="G$1" pin="V_BATT"/>
 <pinref part="C4" gate="G$1" pin="1"/>
-<wire x1="370.84" y1="246.38" x2="370.84" y2="243.84" width="0.1524" layer="91"/>
+<wire x1="365.76" y1="243.84" x2="365.76" y2="241.3" width="0.1524" layer="91"/>
 </segment>
 </net>
@@
 <pinref part="U4" gate="U1" pin="SDA"/>
 <pinref part="FG_SDA" gate="G$1" pin="1"/>
-<wire x1="406.4" y1="241.3" x2="408.94" y2="241.3" width="0.1524" layer="91"/>
-</segment>
-</net>
+<wire x1="401.32" y1="238.76" x2="403.86" y2="238.76" width="0.1524" layer="91"/>
+</segment>
+</net>
