File: Hardware/SparkX_smol_LiPo_Power.brd (EAGLE design)
At the start: 10.7 x 40.6 mm, 54 parts, among them J3 AVR_SPI_PROG_3X2TESTPOINTS, Q1 3.1A/30V/105mΩ, U1 STLQ015-3.3V, U2 MCP73831, U3 3.3V, U4 MAX17048, U5 ATTINY841-ARDUINO_QFN20M1

Commit message: Update smol symbol
Parts:
- added U$3, U$9: SMOL_LOGOSMALL, SparkX:SMOL_SMALL
- moved U$17 0.06 mm to (5.33, 4.57)
Changed lines of the file:
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@@
 <wire x1="7.112" y1="32.639" x2="8.128" y2="32.639" width="0.2032" layer="21"/>
 <wire x1="7.62" y1="32.131" x2="7.62" y2="33.147" width="0.2032" layer="21"/>
-<polygon width="0.0762" layer="21">
-<vertex x="5.334" y="6.096"/>
-<vertex x="2.794" y="5.08"/>
-<vertex x="2.54" y="5.08"/>
-<vertex x="4.572" y="6.858"/>
-<vertex x="6.096" y="6.858"/>
-<vertex x="8.128" y="5.08"/>
-<vertex x="7.874" y="5.08"/>
-</polygon>
-<polygon width="0.0762" layer="22">
-<vertex x="5.334" y="35.687"/>
-<vertex x="7.874" y="34.671"/>
-<vertex x="8.128" y="34.671"/>
-<vertex x="6.096" y="36.449"/>
-<vertex x="4.572" y="36.449"/>
-<vertex x="2.54" y="34.671"/>
-<vertex x="2.794" y="34.671"/>
-</polygon>
 </plain>
 <attributes>
@@
 <element name="U$11" library="output" package="MAX0" value="" x="9.2075" y="30.988" smashed="yes"/>
 <element name="U$8" library="output" package="IN0" value="" x="5.334" y="34.4805" smashed="yes" rot="MR0"/>
-<element name="U$17" library="output" package="OUT0" value="" x="5.334" y="4.6355" smashed="yes"/>
+<element name="U$17" library="output" package="OUT0" value="" x="5.334" y="4.572" smashed="yes"/>
 <element name="U$18" library="output" package="SM�L_POWER_LIPO0" value="" x="9.652" y="9.4615" smashed="yes" rot="R90"/>
 <element name="U$2" library="output" package="SM�L_POWER_LIPO0" value="" x="5.334" y="23.368" smashed="yes" rot="MR0"/>
+<element name="U$3" library="SparkX" package="SMOL_SMALL" value="SMOL_LOGOSMALL" x="5.334" y="6.4135" smashed="yes"/>
+<element name="U$9" library="SparkX" package="SMOL_SMALL" value="SMOL_LOGOSMALL" x="5.334" y="35.814" smashed="yes" rot="MR0"/>
 </elements>
 <signals>
