File: Hardware/Production/SparkX_smol_LiPo_Power-Panel.brd (EAGLE design)
At the start: 198.4 x 137.2 mm, 2502 parts, among them J10 AVR_SPI_PROG_3X2TESTPOINTS, J12 AVR_SPI_PROG_3X2TESTPOINTS, J14 AVR_SPI_PROG_3X2TESTPOINTS, J16 AVR_SPI_PROG_3X2TESTPOINTS, J18 AVR_SPI_PROG_3X2TESTPOINTS, J20 AVR_SPI_PROG_3X2TESTPOINTS, J22 AVR_SPI_PROG_3X2TESTPOINTS, J24 AVR_SPI_PROG_3X2TESTPOINTS, J26 AVR_SPI_PROG_3X2TESTPOINTS, J28 AVR_SPI_PROG_3X2TESTPOINTS, J3 AVR_SPI_PROG_3X2TESTPOINTS, J30 AVR_SPI_PROG_3X2TESTPOINTS, J32 AVR_SPI_PROG_3X2TESTPOINTS, J34 AVR_SPI_PROG_3X2TESTPOINTS, J36 AVR_SPI_PROG_3X2TESTPOINTS, J38 AVR_SPI_PROG_3X2TESTPOINTS, J4 AVR_SPI_PROG_3X2TESTPOINTS, J40 AVR_SPI_PROG_3X2TESTPOINTS, J42 AVR_SPI_PROG_3X2TESTPOINTS, J44 AVR_SPI_PROG_3X2TESTPOINTS, J46 AVR_SPI_PROG_3X2TESTPOINTS, J48 AVR_SPI_PROG_3X2TESTPOINTS, J50 AVR_SPI_PROG_3X2TESTPOINTS, J52 AVR_SPI_PROG_3X2TESTPOINTS, J54 AVR_SPI_PROG_3X2TESTPOINTS, J56 AVR_SPI_PROG_3X2TESTPOINTS, J58 AVR_SPI_PROG_3X2TESTPOINTS, J6 AVR_SPI_PROG_3X2TESTPOINTS, J60 AVR_SPI_PROG_3X2TESTPOINTS, J62 AVR_SPI_PROG_3X2TESTPOINTS, J64 AVR_SPI_PROG_3X2TESTPOINTS, J66 AVR_SPI_PROG_3X2TESTPOINTS, J68 AVR_SPI_PROG_3X2TESTPOINTS, J70 AVR_SPI_PROG_3X2TESTPOINTS, J72 AVR_SPI_PROG_3X2TESTPOINTS, J74 AVR_SPI_PROG_3X2TESTPOINTS, J76 AVR_SPI_PROG_3X2TESTPOINTS, J78 AVR_SPI_PROG_3X2TESTPOINTS, J8 AVR_SPI_PROG_3X2TESTPOINTS, J80 AVR_SPI_PROG_3X2TESTPOINTS, J82 AVR_SPI_PROG_3X2TESTPOINTS, J84 AVR_SPI_PROG_3X2TESTPOINTS, J86 AVR_SPI_PROG_3X2TESTPOINTS, J88 AVR_SPI_PROG_3X2TESTPOINTS, J90 AVR_SPI_PROG_3X2TESTPOINTS, J92 AVR_SPI_PROG_3X2TESTPOINTS, J94 AVR_SPI_PROG_3X2TESTPOINTS, J96 AVR_SPI_PROG_3X2TESTPOINTS, Q1 3.1A/30V/105mΩ, Q10 3.1A/30V/105mΩ, Q11 3.1A/30V/105mΩ, Q12 3.1A/30V/105mΩ, Q13 3.1A/30V/105mΩ, Q14 3.1A/30V/105mΩ, Q15 3.1A/30V/105mΩ, Q16 3.1A/30V/105mΩ, Q17 3.1A/30V/105mΩ, Q18 3.1A/30V/105mΩ, Q19 3.1A/30V/105mΩ, Q2 3.1A/30V/105mΩ, Q20 3.1A/30V/105mΩ, Q21 3.1A/30V/105mΩ, Q22 3.1A/30V/105mΩ, Q23 3.1A/30V/105mΩ, Q24 3.1A/30V/105mΩ, Q25 3.1A/30V/105mΩ, Q26 3.1A/30V/105mΩ, Q27 3.1A/30V/105mΩ, Q28 3.1A/30V/105mΩ, Q29 3.1A/30V/105mΩ, Q3 3.1A/30V/105mΩ, Q30 3.1A/30V/105mΩ, Q31 3.1A/30V/105mΩ, Q32 3.1A/30V/105mΩ, Q33 3.1A/30V/105mΩ, Q34 3.1A/30V/105mΩ, Q35 3.1A/30V/105mΩ, Q36 3.1A/30V/105mΩ, Q37 3.1A/30V/105mΩ, Q38 3.1A/30V/105mΩ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

Commit message: Update smol symbol
Parts:
- added U$721, U$738, U$755, U$772, U$789, U$806: (no value), output:CHG0
- added U$722, U$739, U$756, U$773, U$790, U$807: (no value), output:#RXD0#0
- added U$723, U$740, U$757, U$774, U$791, U$808: (no value), output:#TXD0#0
- added U$724, U$741, U$758, U$775, U$792, U$809: (no value), output:5#5V0
- added U$725, U$742, U$759, U$776, U$793, U$810: (no value), output:MAX0
- added U$726, U$743, U$760, U$777, U$794, U$811: (no value), output:IN0
- added U$727, U$744, U$761, U$778, U$795, U$812: (no value), output:OUT0
- added U$728, U$729, U$745, U$746, U$762, U$763, U$779, U$780, U$796, U$797, U$813, U$814: (no value), output:SM�L_POWER_LIPO0
- added U$730, U$731, U$747, U$748, U$764, U$765, U$781, U$782, U$798, U$799, U$815, U$816: SMOL_LOGOSMALL, SparkX:SMOL_SMALL
- added U$732, U$733, U$749, U$750, U$766, U$767, U$783, U$784, U$800, U$801: SPARKX-LOGO3, SparkX:SPARKX-SMALL
- added U$734, U$751, U$768, U$785, U$802: (no value), output:#BATT##0
- added U$735, U$752, U$769, U$786, U$803: (no value), output:#VIN#0
- added U$736, U$753, U$770, U$787, U$804: (no value), output:#3V3_EN#0
- added U$737, U$754, U$771, U$788, U$805: (no value), output:#PROC_PWR#0
- U$100, U$235, U$355, U$490, U$610: device output:5#5V0 -> output:SM�L_POWER_LIPO0
- U$101, U$221, U$356, U$476, U$611: value (none) -> SMOL_LOGOSMALL; device output:MAX0 -> SparkX:SMOL_SMALL
- U$102, U$237, U$357, U$492, U$612: value (none) -> SMOL_LOGOSMALL; device output:IN0 -> SparkX:SMOL_SMALL
- U$103, U$223, U$358, U$478, U$613: value (none) -> SPARKX-LOGO3; device output:OUT0 -> SparkX:SPARKX-SMALL
- U$104, U$120, U$239, U$240, U$359, U$375, U$494, U$495, U$614, U$630: value (none) -> SPARKX-LOGO3; device output:SM�L_POWER_LIPO0 -> SparkX:SPARKX-SMALL
- U$105, U$224, U$360, U$479, U$615: device output:SM�L_POWER_LIPO0 -> output:#BATT##0
- U$106, U$242, U$361, U$497, U$616: value SPARKX-LOGO3 -> (none); device SparkX:SPARKX-SMALL -> output:#VIN#0
- U$107, U$226, U$362, U$481, U$617: value SPARKX-LOGO3 -> (none); device SparkX:SPARKX-SMALL -> output:#3V3_EN#0
- U$108, U$363, U$618: device output:#BATT##0 -> output:#PROC_PWR#0
- U$109, U$364, U$619: device output:#VIN#0 -> output:CHG0
- U$110, U$365, U$620: device output:#3V3_EN#0 -> output:#RXD0#0
- U$111, U$366, U$621: device output:#PROC_PWR#0 -> output:#TXD0#0
- U$112, U$367, U$622: device output:CHG0 -> output:5#5V0
- U$113, U$368, U$623: device output:#RXD0#0 -> output:MAX0
- U$114, U$369, U$624: device output:#TXD0#0 -> output:IN0
- U$115, U$370, U$625: device output:5#5V0 -> output:OUT0
- U$116, U$236, U$371, U$491, U$626: device output:MAX0 -> output:SM�L_POWER_LIPO0
- U$117, U$252, U$372, U$507, U$627: device output:IN0 -> output:SM�L_POWER_LIPO0
- U$118, U$238, U$373, U$493, U$628: value (none) -> SMOL_LOGOSMALL; device output:OUT0 -> SparkX:SMOL_SMALL
- U$119, U$135, U$254, U$255, U$374, U$390, U$509, U$510, U$629, U$645: value (none) -> SMOL_LOGOSMALL; device output:SM�L_POWER_LIPO0 -> SparkX:SMOL_SMALL
- U$12, U$138, U$273, U$393, U$528, U$648: value (none) -> SPARKX-LOGO3; device output:#BATT##0 -> SparkX:SPARKX-SMALL
- U$122, U$241, U$377, U$496, U$632: value SPARKX-LOGO3 -> (none); device SparkX:SPARKX-SMALL -> output:#BATT##0
- U$123, U$378, U$633: device output:#BATT##0 -> output:#VIN#0
- U$124, U$379, U$634: device output:#VIN#0 -> output:#3V3_EN#0
- U$125, U$380, U$635: device output:#3V3_EN#0 -> output:#PROC_PWR#0
- U$126, U$381, U$636: device output:#PROC_PWR#0 -> output:CHG0
- U$127, U$382, U$637: device output:CHG0 -> output:#RXD0#0
- U$128, U$383, U$638: device output:#RXD0#0 -> output:#TXD0#0
- U$129, U$384, U$639: device output:#TXD0#0 -> output:5#5V0
- U$13, U$154, U$274, U$409, U$529, U$664: value (none) -> SPARKX-LOGO3; device output:#VIN#0 -> SparkX:SPARKX-SMALL
- U$130, U$385, U$640: device output:5#5V0 -> output:MAX0
- U$131, U$386, U$641: device output:MAX0 -> output:IN0
- U$132, U$387, U$642: device output:IN0 -> output:OUT0
- U$133, U$253, U$388, U$508, U$643: device output:OUT0 -> output:SM�L_POWER_LIPO0
- U$136, U$152, U$271, U$272, U$3, U$391, U$407, U$526, U$527, U$646, U$662, U$9: value SPARKX-LOGO3 -> SMOL_LOGOSMALL; device SparkX:SPARKX-SMALL -> SparkX:SMOL_SMALL
- U$139, U$394, U$649: device output:#VIN#0 -> output:#BATT##0
- U$140, U$395, U$650: device output:#3V3_EN#0 -> output:#VIN#0
- U$141, U$396, U$651: device output:#PROC_PWR#0 -> output:#3V3_EN#0
- U$142, U$397, U$652: device output:CHG0 -> output:#PROC_PWR#0
- U$143, U$398, U$653: device output:#RXD0#0 -> output:CHG0
- U$144, U$399, U$654: device output:#TXD0#0 -> output:#RXD0#0
- U$145, U$400, U$655: device output:5#5V0 -> output:#TXD0#0
- U$146, U$401, U$656: device output:MAX0 -> output:5#5V0
- U$147, U$402, U$657: device output:IN0 -> output:MAX0
- U$148, U$403, U$658: device output:OUT0 -> output:IN0
- U$149, U$285, U$30, U$404, U$540, U$659: device output:SM�L_POWER_LIPO0 -> output:OUT0
- U$151, U$167, U$286, U$287, U$31, U$32, U$406, U$422, U$541, U$542, U$661, U$677: value SPARKX-LOGO3 -> (none); device SparkX:SPARKX-SMALL -> output:SM�L_POWER_LIPO0
- U$153, U$288, U$33, U$408, U$543, U$663: value (none) -> SMOL_LOGOSMALL; device output:#BATT##0 -> SparkX:SMOL_SMALL
- U$155, U$290, U$35, U$410, U$545, U$665: value (none) -> SPARKX-LOGO3; device output:#3V3_EN#0 -> SparkX:SPARKX-SMALL
- U$156, U$411, U$666: device output:#PROC_PWR#0 -> output:#BATT##0
- U$157, U$412, U$667: device output:CHG0 -> output:#VIN#0
- U$158, U$413, U$668: device output:#RXD0#0 -> output:#3V3_EN#0
- U$159, U$414, U$669: device output:#TXD0#0 -> output:#PROC_PWR#0
- U$160, U$415, U$670: device output:5#5V0 -> output:CHG0
- U$161, U$416, U$671: device output:MAX0 -> output:#RXD0#0
- U$162, U$417, U$672: device output:IN0 -> output:#TXD0#0
- U$163, U$418, U$673: device output:OUT0 -> output:5#5V0
- U$164, U$300, U$419, U$45, U$555, U$674: device output:SM�L_POWER_LIPO0 -> output:MAX0
- U$165, U$284, U$29, U$420, U$539, U$675: device output:SM�L_POWER_LIPO0 -> output:IN0
- U$166, U$302, U$421, U$47, U$557, U$676: value SPARKX-LOGO3 -> (none); device SparkX:SPARKX-SMALL -> output:OUT0
- U$168, U$303, U$423, U$48, U$558, U$678: device output:#BATT##0 -> output:SM�L_POWER_LIPO0
- U$169, U$289, U$34, U$424, U$544, U$679: value (none) -> SMOL_LOGOSMALL; device output:#VIN#0 -> SparkX:SMOL_SMALL
- U$170, U$305, U$425, U$50, U$560, U$680: value (none) -> SMOL_LOGOSMALL; device output:#3V3_EN#0 -> SparkX:SMOL_SMALL
- U$171, U$291, U$36, U$426, U$546, U$681: value (none) -> SPARKX-LOGO3; device output:#PROC_PWR#0 -> SparkX:SPARKX-SMALL
- U$172, U$307, U$427, U$52, U$562, U$682: value (none) -> SPARKX-LOGO3; device output:CHG0 -> SparkX:SPARKX-SMALL
- U$173, U$428, U$683: device output:#RXD0#0 -> output:#BATT##0
- U$174, U$429, U$684: device output:#TXD0#0 -> output:#VIN#0
- U$175, U$430, U$685: device output:5#5V0 -> output:#3V3_EN#0
- U$176, U$431, U$686: device output:MAX0 -> output:#PROC_PWR#0
- U$177, U$432, U$687: device output:IN0 -> output:CHG0
- U$178, U$433, U$688: device output:OUT0 -> output:#RXD0#0
- U$179, U$315, U$434, U$570, U$60, U$689: device output:SM�L_POWER_LIPO0 -> output:#TXD0#0
- U$180, U$299, U$435, U$44, U$554, U$690: device output:SM�L_POWER_LIPO0 -> output:5#5V0
- U$181, U$317, U$436, U$572, U$62, U$691: value SPARKX-LOGO3 -> (none); device SparkX:SPARKX-SMALL -> output:MAX0
- U$182, U$301, U$437, U$46, U$556, U$692: value SPARKX-LOGO3 -> (none); device SparkX:SPARKX-SMALL -> output:IN0
- U$183, U$438, U$693: device output:#BATT##0 -> output:OUT0
- U$184, U$304, U$439, U$49, U$559, U$694: device output:#VIN#0 -> output:SM�L_POWER_LIPO0
- U$185, U$320, U$440, U$575, U$65, U$695: device output:#3V3_EN#0 -> output:SM�L_POWER_LIPO0
- U$186, U$306, U$441, U$51, U$561, U$696: value (none) -> SMOL_LOGOSMALL; device output:#PROC_PWR#0 -> SparkX:SMOL_SMALL
- U$187, U$322, U$442, U$577, U$67, U$697: value (none) -> SMOL_LOGOSMALL; device output:CHG0 -> SparkX:SMOL_SMALL
- U$188, U$308, U$443, U$53, U$563, U$698: value (none) -> SPARKX-LOGO3; device output:#RXD0#0 -> SparkX:SPARKX-SMALL
- U$189, U$324, U$444, U$579, U$69, U$699: value (none) -> SPARKX-LOGO3; device output:#TXD0#0 -> SparkX:SPARKX-SMALL
- U$19, U$275, U$530: device output:#3V3_EN#0 -> output:#BATT##0
- U$190, U$445, U$700: device output:5#5V0 -> output:#BATT##0
- U$191, U$446, U$701: device output:MAX0 -> output:#VIN#0
- U$192, U$447, U$702: device output:IN0 -> output:#3V3_EN#0
- U$193, U$448, U$703: device output:OUT0 -> output:#PROC_PWR#0
- U$194, U$330, U$449, U$585, U$704, U$75: device output:SM�L_POWER_LIPO0 -> output:CHG0
- U$195, U$314, U$450, U$569, U$59, U$705: device output:SM�L_POWER_LIPO0 -> output:#RXD0#0
- U$196, U$332, U$451, U$587, U$706, U$77: value SPARKX-LOGO3 -> (none); device SparkX:SPARKX-SMALL -> output:#TXD0#0
- U$197, U$316, U$452, U$571, U$61, U$707: value SPARKX-LOGO3 -> (none); device SparkX:SPARKX-SMALL -> output:5#5V0
- U$198, U$453, U$708: device output:#BATT##0 -> output:MAX0
- U$199, U$454, U$709: device output:#VIN#0 -> output:IN0
- U$200, U$455, U$710: device output:#3V3_EN#0 -> output:OUT0
- U$201, U$321, U$456, U$576, U$66, U$711: device output:#PROC_PWR#0 -> output:SM�L_POWER_LIPO0
- U$202, U$337, U$457, U$592, U$712, U$82: device output:CHG0 -> output:SM�L_POWER_LIPO0
- U$203, U$323, U$458, U$578, U$68, U$713: value (none) -> SMOL_LOGOSMALL; device output:#RXD0#0 -> SparkX:SMOL_SMALL
- U$204, U$339, U$459, U$594, U$714, U$84: value (none) -> SMOL_LOGOSMALL; device output:#TXD0#0 -> SparkX:SMOL_SMALL
- U$205, U$325, U$460, U$580, U$70, U$715: value (none) -> SPARKX-LOGO3; device output:5#5V0 -> SparkX:SPARKX-SMALL
- U$206, U$341, U$461, U$596, U$716, U$86: value (none) -> SPARKX-LOGO3; device output:MAX0 -> SparkX:SPARKX-SMALL
- U$207, U$462, U$717: device output:IN0 -> output:#BATT##0
- U$208, U$463, U$718: device output:OUT0 -> output:#VIN#0
- U$209, U$345, U$464, U$600, U$719, U$90: device output:SM�L_POWER_LIPO0 -> output:#3V3_EN#0
- U$21, U$276, U$531: device output:#PROC_PWR#0 -> output:#VIN#0
- U$210, U$329, U$465, U$584, U$720, U$74: device output:SM�L_POWER_LIPO0 -> output:#PROC_PWR#0
- U$211, U$347, U$466, U$602, U$92: value SPARKX-LOGO3 -> (none); device SparkX:SPARKX-SMALL -> output:CHG0
- U$212, U$331, U$467, U$586, U$76: value SPARKX-LOGO3 -> (none); device SparkX:SPARKX-SMALL -> output:#RXD0#0
- U$213, U$468: device output:#BATT##0 -> output:#TXD0#0
- U$214, U$469: device output:#VIN#0 -> output:5#5V0
- U$215, U$470: device output:#3V3_EN#0 -> output:MAX0
- U$216, U$471: device output:#PROC_PWR#0 -> output:IN0
- U$217, U$472: device output:CHG0 -> output:OUT0
- U$218, U$338, U$473, U$593, U$83: device output:#RXD0#0 -> output:SM�L_POWER_LIPO0
- U$219, U$354, U$474, U$609, U$99: device output:#TXD0#0 -> output:SM�L_POWER_LIPO0
- U$22, U$277, U$532: device output:CHG0 -> output:#3V3_EN#0
- U$220, U$340, U$475, U$595, U$85: value (none) -> SMOL_LOGOSMALL; device output:5#5V0 -> SparkX:SMOL_SMALL
- U$222, U$342, U$477, U$597, U$87: value (none) -> SPARKX-LOGO3; device output:IN0 -> SparkX:SPARKX-SMALL
- U$225, U$344, U$480, U$599, U$89: device output:SM�L_POWER_LIPO0 -> output:#VIN#0
- U$227, U$346, U$482, U$601, U$91: value SPARKX-LOGO3 -> (none); device SparkX:SPARKX-SMALL -> output:#PROC_PWR#0
- U$228, U$483: device output:#BATT##0 -> output:CHG0
- U$229, U$484: device output:#VIN#0 -> output:#RXD0#0
- U$23, U$278, U$533: device output:#RXD0#0 -> output:#PROC_PWR#0
- U$230, U$485: device output:#3V3_EN#0 -> output:#TXD0#0
- U$231, U$486: device output:#PROC_PWR#0 -> output:5#5V0
- U$232, U$487: device output:CHG0 -> output:MAX0
- U$233, U$488: device output:#RXD0#0 -> output:IN0
- U$234, U$489: device output:#TXD0#0 -> output:OUT0
- U$24, U$279, U$534: device output:#TXD0#0 -> output:CHG0
- U$243, U$498: device output:#BATT##0 -> output:#3V3_EN#0
- U$244, U$499: device output:#VIN#0 -> output:#PROC_PWR#0
- U$245, U$500: device output:#3V3_EN#0 -> output:CHG0
- U$246, U$501: device output:#PROC_PWR#0 -> output:#RXD0#0
- U$247, U$502: device output:CHG0 -> output:#TXD0#0
- U$248, U$503: device output:#RXD0#0 -> output:5#5V0
- U$249, U$504: device output:#TXD0#0 -> output:MAX0
- U$25, U$280, U$535: device output:5#5V0 -> output:#RXD0#0
- U$250, U$505: device output:5#5V0 -> output:IN0
- U$251, U$506: device output:MAX0 -> output:OUT0
- U$26, U$281, U$536: device output:MAX0 -> output:#TXD0#0
- U$27, U$282, U$537: device output:IN0 -> output:5#5V0
- U$28, U$283, U$538: device output:OUT0 -> output:MAX0
- U$292, U$37, U$547: device output:CHG0 -> output:#BATT##0
- U$293, U$38, U$548: device output:#RXD0#0 -> output:#VIN#0
- U$294, U$39, U$549: device output:#TXD0#0 -> output:#3V3_EN#0
- U$295, U$40, U$550: device output:5#5V0 -> output:#PROC_PWR#0
- U$296, U$41, U$551: device output:MAX0 -> output:CHG0
- U$297, U$42, U$552: device output:IN0 -> output:#RXD0#0
- U$298, U$43, U$553: device output:OUT0 -> output:#TXD0#0
- U$309, U$54, U$564: device output:#TXD0#0 -> output:#BATT##0
- U$310, U$55, U$565: device output:5#5V0 -> output:#VIN#0
- U$311, U$56, U$566: device output:MAX0 -> output:#3V3_EN#0
- U$312, U$567, U$57: device output:IN0 -> output:#PROC_PWR#0
- U$313, U$568, U$58: device output:OUT0 -> output:CHG0
- U$318, U$573, U$63: device output:#BATT##0 -> output:IN0
- U$319, U$574, U$64: device output:#VIN#0 -> output:OUT0
- U$326, U$581, U$71: device output:MAX0 -> output:#BATT##0
- U$327, U$582, U$72: device output:IN0 -> output:#VIN#0
- U$328, U$583, U$73: device output:OUT0 -> output:#3V3_EN#0
- U$333, U$588, U$78: device output:#BATT##0 -> output:5#5V0
- U$334, U$589, U$79: device output:#VIN#0 -> output:MAX0
- U$335, U$590, U$80: device output:#3V3_EN#0 -> output:IN0
- U$336, U$591, U$81: device output:#PROC_PWR#0 -> output:OUT0
- U$343, U$598, U$88: device output:OUT0 -> output:#BATT##0
- U$348, U$603, U$93: device output:#BATT##0 -> output:#RXD0#0
- U$349, U$604, U$94: device output:#VIN#0 -> output:#TXD0#0
- U$350, U$605, U$95: device output:#3V3_EN#0 -> output:5#5V0
- U$351, U$606, U$96: device output:#PROC_PWR#0 -> output:MAX0
- U$352, U$607, U$97: device output:CHG0 -> output:IN0
- U$353, U$608, U$98: device output:#RXD0#0 -> output:OUT0
- moved U$252 173.9 mm to (166.1, 9.46), flipped to the top, turned to 90 degrees
- moved U$243 173.5 mm to (163.5, 7.62)
- moved U$244 171.4 mm to (160.9, 3.75)
- moved U$247 170.7 mm to (164.6, 16.5), flipped to the bottom, turned to 0 degrees
- moved U$251 166.9 mm to (161.8, 4.57)
- moved U$248 166.1 mm to (165.7, 31.9), flipped to the top, turned to 0 degrees
- moved U$268 161.8 mm to (173.0, 4.57)
- moved U$256 161.8 mm to (169.1, 14.1)
- moved U$257 161.8 mm to (173.0, 25.4)
- moved U$258 161.8 mm to (170.9, 33.0)
- moved U$259 161.8 mm to (170.6, 29.2)
- moved U$260 161.8 mm to (174.7, 7.62)
- moved U$261 161.8 mm to (172.1, 3.75)
- moved U$262 161.8 mm to (168.2, 22.7)
- moved U$263 161.8 mm to (169.2, 16.5)
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